File: 65/friendly_Split-65-KiCad/friendly_Split-65.kicad_pcb (KiCad board)
At the start: 2 copper layers, 304.8 x 95.2 mm, 234 parts, among them K1 KEYSW, K10 KEYSW, K11 KEYSW, K12 KEYSW, K13 KEYSW, K14 KEYSW, K15 KEYSW, K16 KEYSW, K17 KEYSW, K18 KEYSW, K19 KEYSW, K2 KEYSW, K20 KEYSW, K21 KEYSW, K22 KEYSW, K23 KEYSW, K24 KEYSW, K25 KEYSW, K26 KEYSW, K27 KEYSW, K28 KEYSW, K29 KEYSW, K3 KEYSW, K30 KEYSW, K31 KEYSW, K32 KEYSW, K33 KEYSW, K34 KEYSW, K35 KEYSW, K36 KEYSW, K37 KEYSW, K38 KEYSW, K39 KEYSW, K4 KEYSW, K40 KEYSW, K41 KEYSW, K42 KEYSW, K43 KEYSW, K44 KEYSW, K45 KEYSW, K46 KEYSW, K47 KEYSW, K48 KEYSW, K49 KEYSW, K5 KEYSW, K50 KEYSW, K51 KEYSW, K52 KEYSW, K53 KEYSW, K54 KEYSW, K55 KEYSW, K56 KEYSW, K57 KEYSW, K58 KEYSW, K59 KEYSW, K6 KEYSW, K60 KEYSW, K61 KEYSW, K62 KEYSW, K63 KEYSW, K64 KEYSW, K65 KEYSW, K66 KEYSW, K67 KEYSW, K68 KEYSW, K69 KEYSW, K7 KEYSW, K70 KEYSW, K71 KEYSW, K8 KEYSW, K9 KEYSW, U2_R1 nice_nano

Commit message: adding the schematics to project
Connections:
- net GND renamed +5V

Commit message: pcb done
Parts:
- removed BT1_L1, BT_R1: 3.7V, Connector_JST:JST_PH_S2B-PH-K_1x02_P2.00mm_Horizontal
- removed D100, D101, D102, D72, D73, D74, D75, D76, D77, D78, D79, D80, D81, D82, D83, D84, D85, D86, D87, D88, D89, D90, D91, D92, D93, D94, D95, D96, D97, D98, D99: D, Diode_SMD:D_SOD-123
- removed D103, D104, D105, D106, D107, D108, D109, D110, D111, D112, D113, D114, D115, D116, D117, D118, D119, D120, D121, D122, D123, D124, D125, D126, D127, D128, D129, D130, D131, D132, D133, D134, D135, D136, D137, D138, D139, D140, D141, D142: SK6805, LED_SMD:LED_SK6805_PLCC4_2.4x2.7mm_P1.3mm
- removed the REF** at (188.1, 114.3)
- removed the REF** at (307.2, 66.7)
- removed the REF** at (238.7, 82.0)
- removed the REF** at (300.0, 38.1)
- removed the REF** at (140.5, 114.3)
- removed the REF** at (106.1, 82.2)
- removed SW_LED_L1, SW_LED_R1: SW_SPDT, Button_Switch_SMD:SW_SPDT_PCM12
- removed U_L1: nice_nano, nice-nano-kicad:nice_nano_mod
- removed the mouse-bite-2mm-slot at (157.2, 57.1)
- removed the mouse-bite-2mm-slot at (161.9, 76.2)
- removed the mouse-bite-2mm-slot at (161.9, 114.3)
- removed the mouse-bite-2mm-slot at (166.7, 38.1)
- removed the mouse-bite-2mm-slot at (171.4, 95.2)
- added BT1: Battery_Cell, Connector_JST:JST_PH_S2B-PH-K_1x02_P2.00mm_Horizontal, F.Cu at (65.5, 30.0)
- added BT2: Battery_Cell, Connector_JST:JST_PH_S2B-PH-K_1x02_P2.00mm_Horizontal, F.Cu at (296.4, 28.0)
- added REF**: M2.5 screw hole, friendly_Split:M2.5 screw hole, F.Cu at (329.4, 46.6)
- added REF**: friendly_Split-logo, friendly_Split:friendly_Split-logo, B.Cu at (93.0, 85.0)
- added REF**: friendly_Split-logo, friendly_Split:friendly_Split-logo, F.Cu at (117.5, 35.5)
- added REF**: M2.5 screw hole, friendly_Split:M2.5 screw hole, F.Cu at (161.2, 138.9)
- added REF**: M2.5 screw hole, friendly_Split:M2.5 screw hole, F.Cu at (153.2, 138.9)
- added REF**: M2.5 screw hole, friendly_Split:M2.5 screw hole, F.Cu at (165.9, 46.6)
- added REF**: M2.5 screw hole, friendly_Split:M2.5 screw hole, F.Cu at (32.6, 46.6)
- added REF**: M2.5 screw hole, friendly_Split:M2.5 screw hole, F.Cu at (157.9, 46.6)
- added REF**: friendly_Split-logo, friendly_Split:friendly_Split-logo, F.Cu at (225.0, 36.0)
- added REF**: friendly_Split-logo, friendly_Split:friendly_Split-logo, B.Cu at (229.5, 84.5)
- added REFe: Lowprofile_Stabilizer_2.00u, friendly_Split:Lowprofile_Stabilizer_2.00u, F.Cu at (135.7, 133.3)
- added REFe: Lowprofile_Stabilizer_2.00u, friendly_Split:Lowprofile_Stabilizer_2.00u, F.Cu at (302.4, 85.7)
- added REFe: Lowprofile_Stabilizer_2.00u, friendly_Split:Lowprofile_Stabilizer_2.00u, F.Cu at (184.0, 133.1)
- added REFe: Lowprofile_Stabilizer_2.00u, friendly_Split:Lowprofile_Stabilizer_2.00u, F.Cu at (295.3, 57.1)
- added U1_L1: nice_nano, nice-nano-kicad:nice_nano, F.Cu at (47.6, 34.6)
- added mouse-bite-2mm-slot: VAL**, Panelization:mouse-bite-2mm-slot, F.Cu at (200.0, 47.6)
- added mouse-bite-2mm-slot: VAL**, Panelization:mouse-bite-2mm-slot, F.Cu at (104.8, 47.6)
- added mouse-bite-2mm-slot: VAL**, Panelization:mouse-bite-2mm-slot, F.Cu at (165.9, 42.6)
- added mouse-bite-2mm-slot: VAL**, Panelization:mouse-bite-2mm-slot, F.Cu at (157.2, 133.3)
- added mouse-bite-2mm-slot: VAL**, Panelization:mouse-bite-2mm-slot, F.Cu at (85.7, 47.6)
- added mouse-bite-2mm-slot: VAL**, Panelization:mouse-bite-2mm-slot, F.Cu at (181.0, 47.6)
- added mouse-bite-2mm-slot: VAL**, Panelization:mouse-bite-2mm-slot, F.Cu at (161.9, 32.6)
- added mouse-bite-2mm-slot: VAL**, Panelization:mouse-bite-2mm-slot, F.Cu at (161.9, 57.1)
- added mouse-bite-2mm-slot: VAL**, Panelization:mouse-bite-2mm-slot, F.Cu at (74.6, 35.6)
- added mouse-bite-2mm-slot: VAL**, Panelization:mouse-bite-2mm-slot, F.Cu at (287.4, 35.6)
- added mouse-bite-2mm-slot: VAL**, Panelization:mouse-bite-2mm-slot, F.Cu at (219.1, 47.6)
- added mouse-bite-2mm-slot: VAL**, Panelization:mouse-bite-2mm-slot, F.Cu at (157.2, 95.2)
- added mouse-bite-2mm-slot: VAL**, Panelization:mouse-bite-2mm-slot, F.Cu at (238.1, 47.6)
- added mouse-bite-2mm-slot: VAL**, Panelization:mouse-bite-2mm-slot, F.Cu at (276.2, 47.6)
- added mouse-bite-2mm-slot: VAL**, Panelization:mouse-bite-2mm-slot, F.Cu at (142.9, 47.6)
- added mouse-bite-2mm-slot: VAL**, Panelization:mouse-bite-2mm-slot, F.Cu at (123.8, 47.6)
- added mouse-bite-2mm-slot: VAL**, Panelization:mouse-bite-2mm-slot, F.Cu at (257.2, 47.6)
- added mouse-bite-2mm-slot: VAL**, Panelization:mouse-bite-2mm-slot, F.Cu at (166.7, 114.3)
- added mouse-bite-2mm-slot: VAL**, Panelization:mouse-bite-2mm-slot, F.Cu at (157.9, 42.6)
- added mouse-bite-2mm-slot: VAL**, Panelization:mouse-bite-2mm-slot, F.Cu at (152.4, 76.2)
- D1, D10, D11, D12, D13, D14, D15, D16, D17, D18, D19, D2, D20, D21, D22, D23, D24, D25, D26, D27, D28, D29, D3, D30, D31, D4, D5, D6, D63, D64, D65, D66, D67, D68, D69, D7, D70, D71, D8, D9: footprint Diode_SMD:D_SOD-123 -> Diode_SMD:D_SMA
- D32, D33, D34, D35, D36, D37, D38, D39, D40, D41, D42, D43, D44, D45, D46, D47, D48, D49, D50, D51, D52, D53, D54, D55, D56, D57, D58, D59, D60, D61, D62: value SK6805 -> D; footprint LED_SMD:LED_SK6805_PLCC4_2.4x2.7mm_P1.3mm -> Diode_SMD:D_SMA; moved to B.Cu
- K1, K10, K11, K12, K13, K15, K16, K17, K18, K19, K2, K21, K22, K23, K24, K25, K26, K28, K3, K30, K32, K33, K34, K35, K36, K37, K39, K4, K40, K41, K42, K43, K44, K45, K46, K48, K49, K5, K50, K51, K52, K53, K54, K55, K56, K57, K58, K59, K6, K60, K61, K63, K64, K67, K69, K7, K70, K71, K9: value KEYSW -> ~; footprint PCM_Switch_Keyboard_Kailh:SW_Kailh_Choc_V1V2_1.00u -> PCM_Switch_Keyboard_Hotswap_Kailh:SW_Hotswap_Kailh_Choc_V1V2_1.00u
- K14, K62: value KEYSW -> ~; footprint PCM_Switch_Keyboard_Kailh:SW_Kailh_Choc_V1V2_1.75u -> PCM_Switch_Keyboard_Hotswap_Kailh:SW_Hotswap_Kailh_Choc_V1V2_1.75u
- K20, K66, K68: value KEYSW -> ~; footprint PCM_Switch_Keyboard_Kailh:SW_Kailh_Choc_V1V2_1.25u -> PCM_Switch_Keyboard_Hotswap_Kailh:SW_Hotswap_Kailh_Choc_V1V2_1.25u
- K27: value KEYSW -> ~; footprint PCM_Switch_Keyboard_Kailh:SW_Kailh_Choc_V1V2_1.50u -> PCM_Switch_Keyboard_Hotswap_Kailh:SW_Hotswap_Kailh_Choc_V1V2_1.25u
- K29: value KEYSW -> ~; footprint PCM_Switch_Keyboard_Kailh:SW_Kailh_Choc_V1V2_1.00u -> PCM_Switch_Keyboard_Hotswap_Kailh:SW_Hotswap_Kailh_Choc_V1V2_1.25u
- K31: value KEYSW -> ~; footprint PCM_Switch_Keyboard_Kailh:SW_Kailh_Choc_V1V2_2.25u -> PCM_Switch_Keyboard_Hotswap_Kailh:SW_Hotswap_Kailh_Choc_V1V2_2.25u
- K38: value KEYSW -> ~; footprint PCM_Switch_Keyboard_Kailh:SW_Kailh_Choc_V1V2_2.00u -> PCM_Switch_Keyboard_Hotswap_Kailh:SW_Hotswap_Kailh_Choc_V1V2_2.00u
- K47: value KEYSW -> ~; footprint PCM_Switch_Keyboard_Kailh:SW_Kailh_Choc_V1V2_ISOEnter_180deg -> PCM_Switch_Keyboard_Hotswap_Kailh:SW_Hotswap_Kailh_Choc_V1V2_ISOEnter
- K65: value KEYSW -> ~; footprint PCM_Switch_Keyboard_Kailh:SW_Kailh_Choc_V1V2_2.75u -> PCM_Switch_Keyboard_Hotswap_Kailh:SW_Hotswap_Kailh_Choc_V1V2_2.75u
- K8: value KEYSW -> ~; footprint PCM_Switch_Keyboard_Kailh:SW_Kailh_Choc_V1V2_1.50u -> PCM_Switch_Keyboard_Hotswap_Kailh:SW_Hotswap_Kailh_Choc_V1V2_1.50u
- SW_PW_L1, SW_PW_R1: moved to F.Cu
- SW_RST_L1, SW_RST_R1: footprint digikey-footprints:Switch_Tactile_SMD_B3U-1000P -> Button_Switch_SMD:SW_Push_1P1T-SH_NO_CK_KMR2xxG; moved to F.Cu
- U2_R1: footprint nice-nano-kicad:nice_nano_mod -> nice-nano-kicad:nice_nano; moved to F.Cu
- moved D39 270.0 mm to (317.6, 52.6)
- moved D47 216.4 mm to (310.9, 88.7), turned to 90 degrees
- moved D45 215.8 mm to (265.7, 79.2), turned to 90 degrees
- moved D46 208.7 mm to (284.7, 79.2), turned to 90 degrees
- moved D48 203.8 mm to (318.1, 70.1), turned to 0 degrees
- moved D56 176.2 mm to (319.1, 90.1)
- moved D51 168.2 mm to (213.3, 98.2), turned to 90 degrees
- moved D52 165.8 mm to (232.3, 98.2), turned to 90 degrees
- moved D54 165.8 mm to (270.4, 98.2), turned to 90 degrees
- moved D55 165.8 mm to (289.5, 98.2), turned to 90 degrees
- moved D53 165.8 mm to (251.4, 98.2), turned to 90 degrees
- moved D71 163.1 mm to (320.1, 128.6), turned to 0 degrees
- moved D58 156.3 mm to (203.8, 117.3), turned to 90 degrees
- moved D60 151.6 mm to (241.9, 117.3), turned to 90 degrees
- moved D61 151.6 mm to (260.9, 117.3), turned to 90 degrees
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Connections:
- D32 pad 1: Net-(D32-DOUT) -> Row0_R
- D32 pad 2: +5V -> Net-(D32-A)
- D33 pad 1: Net-(D33-DOUT) -> Row0_R
- D33 pad 2: +5V -> Net-(D33-A)
- D34 pad 1: Net-(D34-DOUT) -> Row0_R
- D34 pad 2: +5V -> Net-(D34-A)
- D35 pad 1: Net-(D35-DOUT) -> Row0_R
- D35 pad 2: +5V -> Net-(D35-A)
- D36 pad 1: Net-(D36-DOUT) -> Row0_R
- D36 pad 2: +5V -> Net-(D36-A)
- D37 pad 1: Net-(D37-DOUT) -> Row0_R
- D37 pad 2: +5V -> Net-(D37-A)
- D38 pad 1: Net-(D38-DOUT) -> Row0_R
- D38 pad 2: +5V -> Net-(D38-A)
- D39 pad 1: Net-(D39-DOUT) -> Row0_R
- D39 pad 2: +5V -> Net-(D39-A)
- D40 pad 1: Net-(D39-DIN) -> Row1_R
- D40 pad 2: +5V -> Net-(D40-A)
- D41 pad 1: Net-(D40-DIN) -> Row1_R
- D41 pad 2: +5V -> Net-(D41-A)
- D42 pad 1: Net-(D41-DIN) -> Row1_R
- D42 pad 2: +5V -> Net-(D42-A)
- D43 pad 1: Net-(D42-DIN) -> Row1_R
- D43 pad 2: +5V -> Net-(D43-A)
- D44 pad 1: Net-(D43-DIN) -> Row1_R
- D44 pad 2: +5V -> Net-(D44-A)
- D45 pad 1: Net-(D45-DOUT) -> Row1_R
- D45 pad 2: +5V -> Net-(D45-A)
- D46 pad 1: Net-(D46-DOUT) -> Row1_R
- D46 pad 2: +5V -> Net-(D46-A)
- D47 pad 1: Net-(D47-DOUT) -> Row1_R
- D47 pad 2: +5V -> Net-(D47-A)
- D48 pad 1: Net-(D48-DOUT) -> Row1_R
- D48 pad 2: +5V -> Net-(D48-A)
- D49 pad 1: Net-(D49-DOUT) -> Row2_R
- D49 pad 2: +5V -> Net-(D49-A)
- D50 pad 1: Net-(D50-DOUT) -> Row2_R
- D50 pad 2: +5V -> Net-(D50-A)
- D51 pad 1: Net-(D51-DOUT) -> Row2_R
- D51 pad 2: +5V -> Net-(D51-A)
- D52 pad 1: Net-(D51-DIN) -> Row2_R
- D52 pad 2: +5V -> Net-(D52-A)
- D53 pad 1: Net-(D52-DIN) -> Row2_R
- D53 pad 2: +5V -> Net-(D53-A)
- D54 pad 1: Net-(D53-DIN) -> Row2_R
- D54 pad 2: +5V -> Net-(D54-A)
- D55 pad 1: Net-(D54-DIN) -> Row2_R
- D55 pad 2: +5V -> Net-(D55-A)
- D56 pad 1: Net-(D55-DIN) -> Row2_R
- D56 pad 2: +5V -> Net-(D56-A)
- D57 pad 1: Net-(D56-DIN) -> Row3_R
- D57 pad 2: +5V -> Net-(D57-A)
- D58 pad 1: Net-(D58-DOUT) -> Row3_R
- D58 pad 2: +5V -> Net-(D58-A)
- D59 pad 1: Net-(D59-DOUT) -> Row3_R
- D59 pad 2: +5V -> Net-(D59-A)
- D60 pad 1: Net-(D60-DOUT) -> Row3_R
- D60 pad 2: +5V -> Net-(D60-A)
- D61 pad 1: Net-(D61-DOUT) -> Row3_R
- D61 pad 2: +5V -> Net-(D61-A)
- D62 pad 1: unconnected-(D62-DOUT-Pad1) -> Row3_R
- D62 pad 2: +5V -> Net-(D62-A)
- D63 pad 1: Row0_R -> Row3_R
- D64 pad 1: Row0_R -> Row3_R
- D65 pad 1: Row0_R -> Row4_R
- D66 pad 1: Row0_R -> Row4_R
- D67 pad 1: Row0_R -> Row4_R
- D68 pad 1: Row0_R -> Row4_R
- D69 pad 1: Row0_R -> Row4_R
- D70 pad 1: Row0_R -> Row4_R
- D71 pad 1: Row1_R -> Row4_R
- K1 pad 1: Net-(D1-A) -> Col0
- K1 pad 2: Col0 -> Net-(D1-A)
- K10 pad 1: Net-(D10-A) -> Col3
- K10 pad 2: Col3 -> Net-(D10-A)
- K11 pad 1: Net-(D11-A) -> Col4
- K11 pad 2: Col4 -> Net-(D11-A)
- K12 pad 1: Net-(D12-A) -> Col5
- K12 pad 2: Col5 -> Net-(D12-A)
- K13 pad 1: Net-(D13-A) -> Col6
- K13 pad 2: Col6 -> Net-(D13-A)
- K14 pad 1: Net-(D14-A) -> Col0
- K14 pad 2: Col0 -> Net-(D14-A)
- K15 pad 1: Net-(D15-A) -> Col1
- K15 pad 2: Col1 -> Net-(D15-A)
- K16 pad 1: Net-(D16-A) -> Col3
- K16 pad 2: Col3 -> Net-(D16-A)
- K17 pad 1: Net-(D17-A) -> Col4
- K17 pad 2: Col4 -> Net-(D17-A)
- K18 pad 1: Net-(D18-A) -> Col5
- K18 pad 2: Col5 -> Net-(D18-A)
- K19 pad 1: Net-(D19-A) -> Col6
- K19 pad 2: Col6 -> Net-(D19-A)
- K2 pad 1: Net-(D2-A) -> Col1
- K2 pad 2: Col1 -> Net-(D2-A)
- K20 pad 1: Net-(D20-A) -> Col0
- K20 pad 2: Col0 -> Net-(D20-A)
- K21 pad 1: Net-(D21-A) -> Col1
- K21 pad 2: Col1 -> Net-(D21-A)
- K22 pad 1: Net-(D22-A) -> Col2
- K22 pad 2: Col2 -> Net-(D22-A)
- K23 pad 1: Net-(D23-A) -> Col3
- K23 pad 2: Col3 -> Net-(D23-A)
- K24 pad 1: Net-(D24-A) -> Col4
- K24 pad 2: Col4 -> Net-(D24-A)
- K25 pad 1: Net-(D25-A) -> Col5
- K25 pad 2: Col5 -> Net-(D25-A)
- K26 pad 1: Net-(D26-A) -> Col6
- K26 pad 2: Col6 -> Net-(D26-A)
- K27 pad 1: Net-(D27-A) -> Col0
- K27 pad 2: Col0 -> Net-(D27-A)
- K28 pad 1: Net-(D28-A) -> Col1
- K28 pad 2: Col1 -> Net-(D28-A)
- K29 pad 1: Net-(D29-A) -> Col2
- K29 pad 2: Col2 -> Net-(D29-A)
- K3 pad 1: Net-(D3-A) -> Col2
- K3 pad 2: Col2 -> Net-(D3-A)
- K30 pad 1: Net-(D30-A) -> Col3
- K30 pad 2: Col3 -> Net-(D30-A)
- K31 pad 1: Net-(D31-A) -> Col5
- K31 pad 2: Col5 -> Net-(D31-A)
- K32 pad 1: Net-(D63-A) -> Col7
- K32 pad 2: Col7 -> Net-(D32-A)
- K33 pad 1: Net-(D64-A) -> Col8
- K33 pad 2: Col8 -> Net-(D33-A)
- K34 pad 1: Net-(D65-A) -> Col9
- K34 pad 2: Col9 -> Net-(D34-A)
- K35 pad 1: Net-(D66-A) -> Col10
- K35 pad 2: Col10 -> Net-(D35-A)
- K36 pad 1: Net-(D67-A) -> Col11
- K36 pad 2: Col11 -> Net-(D36-A)
- K37 pad 1: Net-(D68-A) -> Col12
- K37 pad 2: Col12 -> Net-(D37-A)
- K38 pad 1: Net-(D69-A) -> Col13
- K38 pad 2: Col13 -> Net-(D38-A)
- K39 pad 1: Net-(D70-A) -> Col15
- K39 pad 2: Col15 -> Net-(D39-A)
- K4 pad 1: Net-(D4-A) -> Col3
- K4 pad 2: Col3 -> Net-(D4-A)
- K40 pad 1: Net-(D71-A) -> Col7
- K40 pad 2: Col7 -> Net-(D40-A)
- K41 pad 1: Net-(D72-A) -> Col8
- K41 pad 2: Col8 -> Net-(D41-A)
- K42 pad 1: Net-(D73-A) -> Col9
- K42 pad 2: Col9 -> Net-(D42-A)
- K43 pad 1: Net-(D74-A) -> Col10
- K43 pad 2: Col10 -> Net-(D43-A)
- K44 pad 1: Net-(D75-A) -> Col11
- K44 pad 2: Col11 -> Net-(D44-A)
- K45 pad 1: Net-(D76-A) -> Col12
- K45 pad 2: Col12 -> Net-(D45-A)
- K46 pad 1: Net-(D77-A) -> Col13
- K46 pad 2: Col13 -> Net-(D46-A)
- K47 pad 1: Net-(D78-A) -> Col14
- K47 pad 2: Col14 -> Net-(D47-A)
- K48 pad 1: Net-(D79-A) -> Col15
- K48 pad 2: Col15 -> Net-(D48-A)
- K49 pad 1: Net-(D80-A) -> Col7
- K49 pad 2: Col7 -> Net-(D49-A)
- K5 pad 1: Net-(D5-A) -> Col4
- K5 pad 2: Col4 -> Net-(D5-A)
- K50 pad 1: Net-(D81-A) -> Col8
- K50 pad 2: Col8 -> Net-(D50-A)
- K51 pad 1: Net-(D82-A) -> Col9
- K51 pad 2: Col9 -> Net-(D51-A)
- K52 pad 1: Net-(D83-A) -> Col10
- K52 pad 2: Col10 -> Net-(D52-A)
- K53 pad 1: Net-(D84-A) -> Col11
- K53 pad 2: Col11 -> Net-(D53-A)
- K54 pad 1: Net-(D85-A) -> Col12
- K54 pad 2: Col12 -> Net-(D54-A)
- K55 pad 1: Net-(D86-A) -> Col13
- K55 pad 2: Col13 -> Net-(D55-A)
- K56 pad 1: Net-(D87-A) -> Col15
- K56 pad 2: Col15 -> Net-(D56-A)
- K57 pad 1: Net-(D88-A) -> Col7
- K57 pad 2: Col7 -> Net-(D57-A)
- K58 pad 1: Net-(D89-A) -> Col8
- K58 pad 2: Col8 -> Net-(D58-A)
- K59 pad 1: Net-(D90-A) -> Col9
- K59 pad 2: Col9 -> Net-(D59-A)
- K6 pad 1: Net-(D6-A) -> Col5
- K6 pad 2: Col5 -> Net-(D6-A)
- K60 pad 1: Net-(D91-A) -> Col10
- K60 pad 2: Col10 -> Net-(D60-A)
- K61 pad 1: Net-(D92-A) -> Col11
- K61 pad 2: Col11 -> Net-(D61-A)
- K62 pad 1: Net-(D93-A) -> Col13
- K62 pad 2: Col13 -> Net-(D62-A)
- K63 pad 1: Net-(D94-A) -> Col14
- K63 pad 2: Col14 -> Net-(D63-A)
- K64 pad 1: Net-(D95-A) -> Col15
- K64 pad 2: Col15 -> Net-(D64-A)
- K65 pad 1: Net-(D96-A) -> Col8
- K65 pad 2: Col8 -> Net-(D65-A)
- K66 pad 1: Net-(D97-A) -> Col9
- K66 pad 2: Col9 -> Net-(D66-A)
- K67 pad 1: Net-(D98-A) -> Col10
- K67 pad 2: Col10 -> Net-(D67-A)
- K68 pad 1: Net-(D99-A) -> Col11
- K68 pad 2: Col11 -> Net-(D68-A)
- K69 pad 1: Net-(D102-A) -> Col13
- K69 pad 2: Col13 -> Net-(D69-A)
- K7 pad 1: Net-(D7-A) -> Col6
- K7 pad 2: Col6 -> Net-(D7-A)
- K70 pad 1: Net-(D100-A) -> Col14
- K70 pad 2: Col14 -> Net-(D70-A)
- K71 pad 1: Net-(D101-A) -> Col15
- K71 pad 2: Col15 -> Net-(D71-A)
- K8 pad 1: Net-(D8-A) -> Col0
- K8 pad 2: Col0 -> Net-(D8-A)
- K9 pad 1: Net-(D9-A) -> Col1
- K9 pad 2: Col1 -> Net-(D9-A)
- SW_PW_L1 pad 2: VBAT_L -> Net-(BT1-+)
- SW_PW_R1 pad 1: unconnected-(SW_PW_R1-A-Pad1) -> Net-(SW_PW_R1-A)
- SW_PW_R1 pad 2: VBAT_R -> Net-(BT2-+)
- SW_PW_R1 pad 3: Net-(SW_PW_R1-C) -> unconnected-(SW_PW_R1-C-Pad3)
- SW_RST_L1 pad 2: +5V -> GND
- SW_RST_R1 pad 2: +5V -> GND
- U2_R1 pad 1: TXD_R -> unconnected-(U2_R1-TX0/P0.06-Pad1)
- U2_R1 pad 10: Col11 -> Col9
- U2_R1 pad 12: Col14 -> Col7
- U2_R1 pad 13: Col13 -> unconnected-(U2_R1-NFC1/P0.09-Pad13)
- U2_R1 pad 14: Col12 -> unconnected-(U2_R1-NFC2/P0.10-Pad14)
- U2_R1 pad 15: unconnected-(U2_R1-P1.11-Pad15) -> Col15
- U2_R1 pad 16: Row1_R -> Row0_R
- U2_R1 pad 17: Row2_R -> Row1_R
- U2_R1 pad 18: Row3_R -> Row2_R
- U2_R1 pad 19: Row4_R -> Row3_R
- U2_R1 pad 20: Row0_R -> Row4_R
- U2_R1 pad 21: Net-(SW_LED_R1-B) -> unconnected-(U2_R1-VCC-Pad21)
- U2_R1 pad 23: +5V -> GND
- U2_R1 pad 24: Net-(SW_PW_R1-C) -> Net-(SW_PW_R1-A)
- U2_R1 pad 3: +5V -> GND
- U2_R1 pad 4: +5V -> GND
- U2_R1 pad 5: Col15 -> Col14
- U2_R1 pad 6: Col7 -> Col13
- U2_R1 pad 7: Col8 -> Col12
- U2_R1 pad 8: Col9 -> Col11
Routing:
- net +5V: track 1587.3 -> 0.00 mm, vias 2 -> 0
- net VCC_LED_R: track 933.5 -> 0.00 mm, vias 3 -> 0
- net VCC_LED_L: track 670.5 -> 0.00 mm, vias 1 -> 0
- net GND: track 0.00 -> 171.3 mm, vias 0 -> 1
- net Col13: track 111.3 -> 197.8 mm, vias 0 -> 2
- net Col11: track 158.3 -> 228.6 mm, vias 0 -> 2
- net Col12: track 99.2 -> 164.1 mm, vias 1 -> 2
- net Col10: track 182.4 -> 245.4 mm
- net Col8: track 226.6 -> 287.5 mm, vias 0 -> 2
- net Net-(D126-DIN): track 56.7 -> 0.00 mm
- net Col9: track 202.7 -> 259.3 mm, vias 0 -> 2
- net Col14: track 85.1 -> 138.1 mm
- net Net-(D136-DIN): track 50.5 -> 0.00 mm
- net VBAT_R: track 48.3 -> 0.00 mm, vias 2 -> 0
- net Col6: track 164.4 -> 208.5 mm, vias 0 -> 4
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Other:
- board size 304.8 x 95.2 mm -> 302.8 x 117.2 mm
- board text added: "V1.1"
- board text removed: "V1.0"
