File: 65/friendly_Split-65-KiCad/friendly_Split-65.kicad_sch (KiCad schematic)
At the start: 0 parts

Commit message: pcb done
Other:
- removed sheet Left
- removed sheet Right
- added sheet left (left.kicad_sch)
- added sheet right (right.kicad_sch)
Changed lines of the file:
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@@
     (rev "V1.0")
   )
-  (sheet (at 156.21 67.31) (size 52.07 57.15) (fields_autoplaced)
+  (sheet (at 156.21 82.55) (size 48.26 41.91) (fields_autoplaced)
     (stroke (width 0.1524) (type solid))
     (fill (color 0 0 0 0.0000))
-    (property "Sheetname" "Right" (at 156.21 66.5984 0)
+    (property "Sheetname" "right" (at 156.21 81.8384 0)
       (effects (font (size 1.27 1.27)) (justify left bottom))
     )
-    (property "Sheetfile" "friendlySplit_right/friendlySplit_right.kicad_sch" (at 156.21 125.0446 0)
+    (property "Sheetfile" "right.kicad_sch" (at 156.21 125.0446 0)
       (effects (font (size 1.27 1.27)) (justify left top))
     )
     (instances
-      (project "friendlySplit"
+      (project "friendly_Split-65"
         (path "/cefbecea-7bec-4164-bd6e-5af8ce6e107d" (page "3"))
       )
     )
   )
-  (sheet (at 64.77 69.85) (size 40.64 53.34) (fields_autoplaced)
+  (sheet (at 66.04 55.245) (size 48.26 55.88) (fields_autoplaced)
     (stroke (width 0.1524) (type solid))
     (fill (color 0 0 0 0.0000))
-    (property "Sheetname" "Left" (at 64.77 69.1384 0)
+    (property "Sheetname" "left" (at 66.04 54.5334 0)
       (effects (font (size 1.27 1.27)) (justify left bottom))
     )
-    (property "Sheetfile" "friendlySplit_left/friendlySplit_left.kicad_sch" (at 64.77 123.7746 0)
+    (property "Sheetfile" "left.kicad_sch" (at 66.04 111.7096 0)
       (effects (font (size 1.27 1.27)) (justify left top))
     )
     (instances
-      (project "friendlySplit"
+      (project "friendly_Split-65"
         (path "/cefbecea-7bec-4164-bd6e-5af8ce6e107d" (page "2"))
       )
